Commit message: beta version after adding reach_target and reach_home

File: assets/urdf/cube.urdf (robot description, URDF)
Before this commit: robot object, 1 links, 0 joints
Links:
- link object: mass 0.5 -> 1.5; geometry collision box size=0.5 0.5 0.5; visual box size=0.5 0.5 0.5

File: assets/urdf/objects/cube_multicolor.urdf (robot description, URDF)
Before this commit: robot object, 1 links, 0 joints
Links:
- link object: geometry collision box size=0.5 0.5 0.5; visual mesh filename=meshes/cube_multicolor.obj scale=.5 .5 .5
